Commit message: renamed package

File: bipedal_description/urdf/bipedal.xacro (robot description, xacro)
@@ -1,7 +1,7 @@
 <?xml version="1.0" ?>
-<robot name="BiPedal" xmlns:xacro="http://www.ros.org/wiki/xacro">
-<xacro:include filename="$(find BiPedal_description)/urdf/materials.xacro" />
-<xacro:include filename="$(find BiPedal_description)/urdf/BiPedal.trans" />
-<xacro:include filename="$(find BiPedal_description)/urdf/BiPedal.gazebo" />
+<robot name="bipedal" xmlns:xacro="http://www.ros.org/wiki/xacro">
+<xacro:include filename="$(find bipedal_description)/urdf/materials.xacro" />
+<xacro:include filename="$(find bipedal_description)/urdf/bipedal.trans" />
+<xacro:include filename="$(find bipedal_description)/urdf/bipedal.gazebo" />
 <link name="base_link">
   <inertial>
@@ -13,5 +13,5 @@
     <origin xyz="0 0 0" rpy="0 0 0"/>
     <geometry>
-      <mesh filename="file://$(find BiPedal_description)/meshes/base_link.stl" scale="0.001 0.001 0.001"/>
+      <mesh filename="file://$(find bipedal_description)/meshes/base_link.stl" scale="0.001 0.001 0.001"/>
     </geometry>
     <material name="silver"/>
@@ -20,5 +20,5 @@
     <origin xyz="0 0 0" rpy="0 0 0"/>
     <geometry>
-      <mesh filename="file://$(find BiPedal_description)/meshes/base_link.stl" scale="0.001 0.001 0.001"/>
+      <mesh filename="file://$(find bipedal_description)/meshes/base_link.stl" scale="0.001 0.001 0.001"/>
     </geometry>
   </collision>
@@ -33,5 +33,5 @@
     <origin xyz="-0.0695 -0.0152 -0.03505" rpy="0 0 0"/>
     <geometry>
-      <mesh filename="file://$(find BiPedal_description)/meshes/l_limb_1_2.stl" scale="0.001 0.001 0.001"/>
+      <mesh filename="file://$(find bipedal_description)/meshes/l_limb_1_2.stl" scale="0.001 0.001 0.001"/>
     </geometry>
     <material name="silver"/>
@@ -40,5 +40,5 @@
     <origin xyz="-0.0695 -0.0152 -0.03505" rpy="0 0 0"/>
     <geometry>
-      <mesh filename="file://$(find BiPedal_description)/meshes/l_limb_1_2.stl" scale="0.001 0.001 0.001"/>
+      <mesh filename="file://$(find bipedal_description)/meshes/l_limb_1_2.stl" scale="0.001 0.001 0.001"/>
     </geometry>
   </collision>
@@ -53,5 +53,5 @@
     <origin xyz="-0.0125 -0.02285 -0.02715" rpy="0 0 0"/>
     <geometry>
-      <mesh filename="file://$(find BiPedal_description)/meshes/l_limb_2_1.stl" scale="0.001 0.001 0.001"/>
+      <mesh filename="file://$(find bipedal_description)/meshes/l_limb_2_1.stl" scale="0.001 0.001 0.001"/>
     </geometry>
     <material name="silver"/>
@@ -60,5 +60,5 @@
     <origin xyz="-0.0125 -0.02285 -0.02715" rpy="0 0 0"/>
     <geometry>
-      <mesh filename="file://$(find BiPedal_description)/meshes/l_limb_2_1.stl" scale="0.001 0.001 0.001"/>
+      <mesh filename="file://$(find bipedal_description)/meshes/l_limb_2_1.stl" scale="0.001 0.001 0.001"/>
     </geometry>
   </collision>
@@ -73,5 +73,5 @@
     <origin xyz="-0.00245 -0.01225 0.013" rpy="0 0 0"/>
     <geometry>
-      <mesh filename="file://$(find BiPedal_description)/meshes/l_limb_3_1.stl" scale="0.001 0.001 0.001"/>
+      <mesh filename="file://$(find bipedal_description)/meshes/l_limb_3_1.stl" scale="0.001 0.001 0.001"/>
     </geometry>
     <material name="silver"/>
@@ -80,5 +80,5 @@
     <origin xyz="-0.00245 -0.01225 0.013" rpy="0 0 0"/>
     <geometry>
-      <mesh filename="file://$(find BiPedal_description)/meshes/l_limb_3_1.stl" scale="0.001 0.001 0.001"/>
+      <mesh filename="file://$(find bipedal_description)/meshes/l_limb_3_1.stl" scale="0.001 0.001 0.001"/>
     </geometry>
   </collision>
@@ -93,5 +93,5 @@
     <origin xyz="-0.00245 -0.01225 0.088" rpy="0 0 0"/>
     <geometry>
-      <mesh filename="file://$(find BiPedal_description)/meshes/l_limb_4_1.stl" scale="0.001 0.001 0.001"/>
+      <mesh filename="file://$(find bipedal_description)/meshes/l_limb_4_1.stl" scale="0.001 0.001 0.001"/>
     </geometry>
     <material name="silver"/>
@@ -100,5 +100,5 @@
     <origin xyz="-0.00245 -0.01225 0.088" rpy="0 0 0"/>
     <geometry>
-      <mesh filename="file://$(find BiPedal_description)/meshes/l_limb_4_1.stl" scale="0.001 0.001 0.001"/>
+      <mesh filename="file://$(find bipedal_description)/meshes/l_limb_4_1.stl" scale="0.001 0.001 0.001"/>
     </geometry>
   </collision>
@@ -113,5 +113,5 @@
     <origin xyz="-0.00245 -0.01225 0.148" rpy="0 0 0"/>
     <geometry>
-      <mesh filename="file://$(find BiPedal_description)/meshes/l_limb_5_1.stl" scale="0.001 0.001 0.001"/>
+      <mesh filename="file://$(find bipedal_description)/meshes/l_limb_5_1.stl" scale="0.001 0.001 0.001"/>
     </geometry>
     <material name="silver"/>
@@ -120,5 +120,5 @@
     <origin xyz="-0.00245 -0.01225 0.148" rpy="0 0 0"/>
     <geometry>
-      <mesh filename="file://$(find BiPedal_description)/meshes/l_limb_5_1.stl" scale="0.001 0.001 0.001"/>
+      <mesh filename="file://$(find bipedal_description)/meshes/l_limb_5_1.stl" scale="0.001 0.001 0.001"/>
     </geometry>
   </collision>
@@ -133,5 +133,5 @@
     <origin xyz="-0.102233 -0.0152 -0.03505" rpy="0 0 0"/>
     <geometry>
-      <mesh filename="file://$(find BiPedal_description)/meshes/r_limb_1_2.stl" scale="0.001 0.001 0.001"/>
+      <mesh filename="file://$(find bipedal_description)/meshes/r_limb_1_2.stl" scale="0.001 0.001 0.001"/>
     </geometry>
     <material name="silver"/>
@@ -140,5 +140,5 @@
     <origin xyz="-0.102233 -0.0152 -0.03505" rpy="0 0 0"/>
     <geometry>
-      <mesh filename="file://$(find BiPedal_description)/meshes/r_limb_1_2.stl" scale="0.001 0.001 0.001"/>
+      <mesh filename="file://$(find bipedal_description)/meshes/r_limb_1_2.stl" scale="0.001 0.001 0.001"/>
     </geometry>
   </collision>
@@ -153,5 +153,5 @@
     <origin xyz="-0.159233 -0.02285 -0.02715" rpy="0 0 0"/>
     <geometry>
-      <mesh filename="file://$(find BiPedal_description)/meshes/r_limb_2_1.stl" scale="0.001 0.001 0.001"/>
+      <mesh filename="file://$(find bipedal_description)/meshes/r_limb_2_1.stl" scale="0.001 0.001 0.001"/>
     </geometry>
     <material name="silver"/>
@@ -160,5 +160,5 @@
     <origin xyz="-0.159233 -0.02285 -0.02715" rpy="0 0 0"/>
     <geometry>
-      <mesh filename="file://$(find BiPedal_description)/meshes/r_limb_2_1.stl" scale="0.001 0.001 0.001"/>
+      <mesh filename="file://$(find bipedal_description)/meshes/r_limb_2_1.stl" scale="0.001 0.001 0.001"/>
     </geometry>
   </collision>
@@ -173,5 +173,5 @@
     <origin xyz="-0.169283 -0.01225 0.013" rpy="0 0 0"/>
     <geometry>
-      <mesh filename="file://$(find BiPedal_description)/meshes/r_limb_3_1.stl" scale="0.001 0.001 0.001"/>
+      <mesh filename="file://$(find bipedal_description)/meshes/r_limb_3_1.stl" scale="0.001 0.001 0.001"/>
     </geometry>
     <material name="silver"/>
@@ -180,5 +180,5 @@
     <origin xyz="-0.169283 -0.01225 0.013" rpy="0 0 0"/>
     <geometry>
-      <mesh filename="file://$(find BiPedal_description)/meshes/r_limb_3_1.stl" scale="0.001 0.001 0.001"/>
+      <mesh filename="file://$(find bipedal_description)/meshes/r_limb_3_1.stl" scale="0.001 0.001 0.001"/>
     </geometry>
   </collision>
@@ -193,5 +193,5 @@
     <origin xyz="-0.169283 -0.01225 0.088" rpy="0 0 0"/>
     <geometry>
-      <mesh filename="file://$(find BiPedal_description)/meshes/r_limb_4_1.stl" scale="0.001 0.001 0.001"/>
+      <mesh filename="file://$(find bipedal_description)/meshes/r_limb_4_1.stl" scale="0.001 0.001 0.001"/>
     </geometry>
     <material name="silver"/>
@@ -200,5 +200,5 @@
     <origin xyz="-0.169283 -0.01225 0.088" rpy="0 0 0"/>
     <geometry>
-      <mesh filename="file://$(find BiPedal_description)/meshes/r_limb_4_1.stl" scale="0.001 0.001 0.001"/>
+      <mesh filename="file://$(find bipedal_description)/meshes/r_limb_4_1.stl" scale="0.001 0.001 0.001"/>
     </geometry>
   </collision>
@@ -213,5 +213,5 @@
     <origin xyz="-0.169283 -0.01225 0.148" rpy="0 0 0"/>
     <geometry>
-      <mesh filename="file://$(find BiPedal_description)/meshes/r_limb_5_1.stl" scale="0.001 0.001 0.001"/>
+      <mesh filename="file://$(find bipedal_description)/meshes/r_limb_5_1.stl" scale="0.001 0.001 0.001"/>
     </geometry>
     <material name="silver"/>
@@ -220,5 +220,5 @@
     <origin xyz="-0.169283 -0.01225 0.148" rpy="0 0 0"/>
     <geometry>
-      <mesh filename="file://$(find BiPedal_description)/meshes/r_limb_5_1.stl" scale="0.001 0.001 0.001"/>
+      <mesh filename="file://$(find bipedal_description)/meshes/r_limb_5_1.stl" scale="0.001 0.001 0.001"/>
     </geometry>
   </collision>

File: bipedal_description/urdf/materials.xacro (robot description, xacro)
@@ -1,4 +1,4 @@
 <?xml version="1.0" ?>
-<robot name="BiPedal" xmlns:xacro="http://www.ros.org/wiki/xacro" >
+<robot name="bipedal" xmlns:xacro="http://www.ros.org/wiki/xacro" >
 <material name="silver">
   <color rgba="0.700 0.700 0.700 1.000"/>
